Commit message: fix resource not found error

File: urdf/kobuki.urdf.xacro (robot description, xacro)
@@ -7,6 +7,6 @@
  -->
 <robot name="kobuki" xmlns:xacro="http://ros.org/wiki/xacro">
-  <xacro:include filename="$(find robot_gazebo)/urdf/common_properties.urdf.xacro"/>
-  <xacro:include filename="$(find robot_gazebo)/urdf/kobuki_gazebo.urdf.xacro"/>
+  <xacro:include filename="$(find followbot)/urdf/common_properties.urdf.xacro"/>
+  <xacro:include filename="$(find followbot)/urdf/kobuki_gazebo.urdf.xacro"/>
   <!-- Kobuki -->
   <xacro:macro name="kobuki">

File: urdf/kobuki_standalone.urdf.xacro (robot description, xacro)
@@ -6,5 +6,5 @@
        xmlns:xacro="http://ros.org/wiki/xacro">
   <!-- Defines the kobuki component tag. -->
-  <xacro:include filename="$(find kobuki_description)/urdf/kobuki.urdf.xacro" />
+  <xacro:include filename="$(find followbot)/urdf/kobuki.urdf.xacro" />
   <kobuki/>
 </robot>

File: urdf/sensors/hokuyo.urdf.xacro (robot description, xacro)
@@ -2,5 +2,5 @@
 <!-- script_version=1.1 -->
 <robot name="sensor_hokuyo" xmlns:xacro="http://ros.org/wiki/xacro">
-  <xacro:include filename="$(find robot_gazebo)/urdf/common_properties.urdf.xacro"/>
+  <xacro:include filename="$(find followbot)/urdf/common_properties.urdf.xacro"/>
   <!-- RPLidar 2D LIDAR -->
   <xacro:macro name="sensor_hokuyo" params="parent">
@@ -21,5 +21,5 @@
       <origin xyz="0 0 0" rpy="0 0 0" />
       <geometry>
-        <mesh filename="package://robot_gazebo/meshes/sensors/hokuyo.dae" />
+        <mesh filename="package://followbot/meshes/sensors/hokuyo.dae" />
       </geometry>
     </visual>

File: urdf/sensors/kinect.urdf.xacro (robot description, xacro)
@@ -1,6 +1,6 @@
 <?xml version="1.0"?>
 <robot name="sensor_kinect" xmlns:xacro="http://ros.org/wiki/xacro">
-  <xacro:include filename="$(find turtlebot_description)/urdf/turtlebot_gazebo.urdf.xacro"/>
-  <xacro:include filename="$(find turtlebot_description)/urdf/turtlebot_properties.urdf.xacro"/>
+  <xacro:include filename="$(find followbot)/urdf/turtlebot_gazebo.urdf.xacro"/>
+  <xacro:include filename="$(find followbot)/urdf/turtlebot_properties.urdf.xacro"/>
   <xacro:property name="kinect_cam_py" value="-0.0125"/>
   <xacro:property name="cam_or" value="0"/>
@@ -30,5 +30,5 @@
        <origin xyz="0 0 0" rpy="0 0 ${M_PI/2}"/>
         <geometry>
-         <mesh filename="package://robot_gazebo/meshes/sensors/kinect.dae"/>
+         <mesh filename="package://followbot/meshes/sensors/kinect.dae"/>
         </geometry>
       </visual>

File: urdf/stacks/hexagons.urdf.xacro (robot description, xacro)
@@ -4,5 +4,5 @@
  -->
 <robot name="stack_hexagons" xmlns:xacro="http://ros.org/wiki/xacro">
-  <xacro:include filename="$(find robot_gazebo)/urdf/common_properties.urdf.xacro"/>
+  <xacro:include filename="$(find followbot)/urdf/common_properties.urdf.xacro"/>
   <!-- Xacro properties -->
   <xacro:property name="M_SCALE" value="0.001"/>

File: urdf/turtlebot_common_library.urdf.xacro (robot description, xacro)
@@ -5,6 +5,6 @@
 <robot xmlns:xacro="http://ros.org/wiki/xacro">
   <!-- General -->
-  <xacro:include filename="$(find robot_gazebo)/urdf/common_properties.urdf.xacro"/>
-  <xacro:include filename="$(find robot_gazebo)/urdf/turtlebot_properties.urdf.xacro"/>
-  <!--<xacro:include filename="$(find robot_gazebo)/urdf/sensors/hokuyo.urdf.xacro"/>-->
+  <xacro:include filename="$(find followbot)/urdf/common_properties.urdf.xacro"/>
+  <xacro:include filename="$(find followbot)/urdf/turtlebot_properties.urdf.xacro"/>
+  <!--<xacro:include filename="$(find followbot)/urdf/sensors/hokuyo.urdf.xacro"/>-->
 </robot>

Commit message: Add rounded corners to the track map and fix some urdf path problem

File: urdf/kobuki.urdf.xacro (robot description, xacro)
@@ -30,5 +30,5 @@
         <geometry>
           <!-- new mesh -->
-          <mesh filename="package://kobuki_description/meshes/main_body.dae" />
+          <mesh filename="package://followbot/meshes/kobuki/main_body.dae" />
         </geometry>
         <origin xyz="0.001 0 0.05199" rpy="0 0 0"/>
@@ -65,5 +65,5 @@
       <visual>
         <geometry>
-          <mesh filename="package://kobuki_description/meshes/wheel.dae"/>
+          <mesh filename="package://followbot/meshes/kobuki/wheel.dae"/>
         </geometry>
         <origin xyz="0 0 0" rpy="0 0 0"/>
@@ -92,5 +92,5 @@
       <visual>
         <geometry>
-          <mesh filename="package://kobuki_description/meshes/wheel.dae"/>
+          <mesh filename="package://followbot/meshes/kobuki/wheel.dae"/>
         </geometry>
         <origin xyz="0 0 0" rpy="0 0 0"/>

File: urdf/sensors/hokuyo.urdf.xacro (robot description, xacro)
@@ -6,5 +6,5 @@
   <xacro:macro name="sensor_hokuyo" params="parent">
     <joint name="laser" type="fixed">
-      <origin xyz="0.1 0 0.45" rpy="0 0.0 0" />
+      <origin xyz="0.1 0 0.43" rpy="0 0.0 0" />
       <parent link="${parent}" />
       <child link="hokuyo_link" />

File: urdf/sensors/kinect.urdf.xacro (robot description, xacro)
@@ -4,11 +4,8 @@
   <xacro:include filename="$(find followbot)/urdf/turtlebot_properties.urdf.xacro"/>
   <xacro:property name="kinect_cam_py" value="-0.0125"/>
-  <xacro:property name="cam_or" value="0"/>
-  <xacro:property name="cam_op" value="${M_PI/2}"/>
-  <xacro:property name="cam_oy" value="0"/>
   <!-- Parameterised in part by the values in turtlebot_properties.urdf.xacro -->
   <xacro:macro name="sensor_kinect" params="parent">
     <joint name="camera_rgb_joint" type="fixed">
-      <origin xyz="0.18 ${kinect_cam_py} 0.19" rpy="${cam_or} ${cam_op} ${cam_oy}"/>
+      <origin xyz="${cam_px} ${kinect_cam_py} ${cam_pz}" rpy="${cam_or} ${cam_op} ${cam_oy}"/>
       <parent link="${parent}"/>
       <child link="camera_rgb_frame" />

File: urdf/stacks/hexagons.urdf.xacro (robot description, xacro)
@@ -19,5 +19,5 @@
         <origin xyz="0 0 0" rpy="0 0 0"/>
         <geometry>
-          <mesh filename="package://turtlebot_description/meshes/stacks/hexagons/pole_bottom.dae"/>
+          <mesh filename="package://followbot/meshes/stacks/hexagons/pole_bottom.dae"/>
         </geometry>
       </visual>
@@ -47,5 +47,5 @@
         <origin xyz="0 0 0" rpy="0 ${M_PI} 0"/>
         <geometry>
-          <mesh filename="package://turtlebot_description/meshes/stacks/hexagons/pole_middle.dae"/>
+          <mesh filename="package://followbot/meshes/stacks/hexagons/pole_middle.dae"/>
         </geometry>
       </visual>
@@ -75,5 +75,5 @@
         <origin xyz=" 0 0 0" rpy="0 0 0"/>
         <geometry>
-          <mesh filename="package://turtlebot_description/meshes/stacks/hexagons/pole_top.dae"/>
+          <mesh filename="package://followbot/meshes/stacks/hexagons/pole_top.dae"/>
         </geometry>
       </visual>
@@ -103,5 +103,5 @@
         <!--<origin xyz="0 0 -0.01" rpy="0 0 0"/>-->
         <!--<geometry>-->
-          <!--<mesh filename="package://turtlebot_description/meshes/sensors/sensor_pole.dae" />-->
+          <!--<mesh filename="package://followbot/meshes/sensors/sensor_pole.dae" />-->
         <!--</geometry>-->
       <!--</visual>-->
@@ -142,5 +142,5 @@
         <origin xyz="0 0 0" rpy="0 0 0"/>
         <geometry>
-          <mesh filename="package://turtlebot_description/meshes/stacks/hexagons/plate_bottom.dae"/>
+          <mesh filename="package://followbot/meshes/stacks/hexagons/plate_bottom.dae"/>
         </geometry>
       </visual>
@@ -172,5 +172,5 @@
         <origin xyz="0 0 0" rpy="0 0 0"/>
         <geometry>
-          <mesh filename="package://turtlebot_description/meshes/stacks/hexagons/plate_middle.dae"/>
+          <mesh filename="package://followbot/meshes/stacks/hexagons/plate_middle.dae"/>
         </geometry>
       </visual>
@@ -204,5 +204,5 @@
         <origin xyz="0 0 0" rpy="0 0 0"/>
         <geometry>
-          <mesh filename="package://turtlebot_description/meshes/stacks/hexagons/plate_top.dae"/>
+          <mesh filename="package://followbot/meshes/stacks/hexagons/plate_top.dae"/>
         </geometry>
       </visual>

File: urdf/turtlebot_properties.urdf.xacro (robot description, xacro)
@@ -19,9 +19,9 @@
      (currently in development and awaiting feedback)
    -->
-	<xacro:property name="cam_px" value="-0.087" />
+	<xacro:property name="cam_px" value="0.18" />
 <!--	<xacro:property name="cam_py" value="-0.0125" /> Y varies for different configurations. get sets in sensors_urdf -->
-	<xacro:property name="cam_pz" value="0.2870" />
-	<xacro:property name="cam_or" value="0" />
-	<xacro:property name="cam_op" value="0" />
-	<xacro:property name="cam_oy" value="0" />
+	<xacro:property name="cam_pz" value="0.19" />
+  <xacro:property name="cam_or" value="0"/>
+  <xacro:property name="cam_op" value="${M_PI/2}"/>
+  <xacro:property name="cam_oy" value="0"/>
 </robot>
