Commit message: Add a monocular camera to the Fred robot

File: urdf/fred/fred_gazebo.urdf.xacro (robot description, xacro)
@@ -6,5 +6,5 @@
       <sensor type="depth" name="camera">
         <always_on>true</always_on>
-        <update_rate>100.0</update_rate>
+        <update_rate>600.0</update_rate>
         <camera>
           <horizontal_fov>${90.0*M_PI/180.0}</horizontal_fov>
@@ -22,5 +22,5 @@
           <cameraName>camera</cameraName>
           <alwaysOn>true</alwaysOn>
-          <updateRate>100</updateRate>
+          <updateRate>600</updateRate>
           <imageTopicName>rgb/image_raw</imageTopicName>
           <depthImageTopicName>depth/image_raw</depthImageTopicName>
@@ -36,4 +36,53 @@
           <distortion_t2>0.0</distortion_t2>
           <pointCloudCutoff>0.0</pointCloudCutoff>
+        </plugin>
+      </sensor>
+    </gazebo>
+  </xacro:macro>
+  <!-- Monocular camera -->
+  <xacro:macro name="fred_sim_2dsensor_cam">
+    <gazebo reference="mono_camera_link">
+      <sensor type="camera" name="mono_camera">
+        <update_rate>30.0</update_rate>
+        <camera name="head">
+          <horizontal_fov>${90.0*M_PI/180.0}</horizontal_fov>
+          <image>
+            <width>1280</width>
+            <height>720</height>
+            <format>R8G8B8</format>
+          </image>
+          <clip>
+            <near>0.02</near>
+            <far>30</far>
+          </clip>
+          <noise>
+            <type>gaussian</type>
+            <!-- Noise is sampled independently per pixel on each frame.
+                That pixel's noise value is added to each of its color
+                channels, which at that point lie in the range [0,1]. -->
+            <mean>0.0</mean>
+            <stddev>0.007</stddev>
+          </noise>
+        </camera>
+        <plugin name="camera_controller" filename="libgazebo_ros_camera.so">
+          <alwaysOn>true</alwaysOn>
+          <updateRate>0.0</updateRate>
+          <cameraName>usb_cam</cameraName>
+          <imageTopicName>image_raw</imageTopicName>
+          <cameraInfoTopicName>camera_info</cameraInfoTopicName>
+          <frameName>mono_camera_optical_frame</frameName>
+          <!-- setting hackBaseline to anything but 0.0 will cause a misalignment
+              between the gazebo sensor image and the frame it is supposed to
+              be attached to -->
+          <hackBaseline>0.07</hackBaseline>
+          <distortionK1>0.0</distortionK1>
+          <distortionK2>0.0</distortionK2>
+          <distortionK3>0.0</distortionK3>
+          <distortionT1>0.0</distortionT1>
+          <distortionT2>0.0</distortionT2>
+          <CxPrime>0</CxPrime>
+          <Cx>0.0</Cx>
+          <Cy>0.0</Cy>
+          <focalLength>0</focalLength>
         </plugin>
       </sensor>

File: urdf/fred/fred_properties.urdf.xacro (robot description, xacro)
@@ -25,4 +25,22 @@
   <xacro:property name="cam_op" value="${M_PI/2}"/>
   <xacro:property name="cam_oy" value="0"/>
+    <!--
+   ======================================================================
+   - REP 119 : Monocular camera link relative to the Base link
+   ======================================================================
+     Base link is currently defined as the rotational centre on the bottom
+     of the base mould. For both create and kobuki this is actually exactly
+     the same 3d world point.
+     This may cause an issue with a base with much different floor clearance.
+     Should we be using base_footprint for this specification instead?
+     Note: REP needs to be updated with the information below
+     (currently in development and awaiting feedback)
+   -->
+	<xacro:property name="mono_cam_px" value="0.68" />
+<!--	<xacro:property name="cam_py" value="-0.0125" /> Y varies for different configurations. get sets in sensors_urdf -->
+	<xacro:property name="mono_cam_pz" value="0.11" />
+  <xacro:property name="mono_cam_or" value="0"/>
+  <xacro:property name="mono_cam_op" value="0"/>
+  <xacro:property name="mono_cam_oy" value="0"/>
   <!--
   ======================================================================

Commit message: Add files via upload

File: urdf/fred/fred_gazebo.urdf.xacro (robot description, xacro)
@@ -6,5 +6,5 @@
       <sensor type="depth" name="camera">
         <always_on>true</always_on>
-        <update_rate>100.0</update_rate>
+        <update_rate>600.0</update_rate>
         <camera>
           <horizontal_fov>${90.0*M_PI/180.0}</horizontal_fov>
@@ -22,5 +22,5 @@
           <cameraName>camera</cameraName>
           <alwaysOn>true</alwaysOn>
-          <updateRate>100</updateRate>
+          <updateRate>600</updateRate>
           <imageTopicName>rgb/image_raw</imageTopicName>
           <depthImageTopicName>depth/image_raw</depthImageTopicName>
@@ -40,4 +40,91 @@
     </gazebo>
   </xacro:macro>
+    <!-- Monocular camera -->
+  <xacro:macro name="fred_sim_2dsensor_cam">
+    <gazebo reference="mono_camera_link">
+      <sensor type="depth" name="mono_camera">
+        <always_on>true</always_on>
+        <update_rate>60.0</update_rate>
+        <camera>
+          <horizontal_fov>${90*M_PI/180.0}</horizontal_fov>
+          <image>
+            <format>B8G8R8</format>
+            <width>640</width>
+            <height>360</height>
+          </image>
+          <clip>
+            <near>0.05</near>
+            <far>8.0</far>
+          </clip>
+        </camera>
+        <plugin name="kinect_camera_controller" filename="libgazebo_ros_openni_kinect.so">
+          <cameraName>usb_cam</cameraName>
+          <alwaysOn>true</alwaysOn>
+          <updateRate>60</updateRate>
+          <imageTopicName>rgb/image_raw</imageTopicName>
+          <depthImageTopicName>depth/image_raw</depthImageTopicName>
+          <pointCloudTopicName>depth/points</pointCloudTopicName>
+          <cameraInfoTopicName>rgb/camera_info</cameraInfoTopicName>
+          <depthImageCameraInfoTopicName>depth/camera_info</depthImageCameraInfoTopicName>
+          <frameName>mono_camera_depth_optical_frame</frameName>
+          <baseline>0.1</baseline>
+          <distortion_k1>0.0</distortion_k1>
+          <distortion_k2>0.0</distortion_k2>
+          <distortion_k3>0.0</distortion_k3>
+          <distortion_t1>0.0</distortion_t1>
+          <distortion_t2>0.0</distortion_t2>
+          <pointCloudCutoff>0.0</pointCloudCutoff>
+        </plugin>
+      </sensor>
+    </gazebo>
+  </xacro:macro>
+<!--  <xacro:macro name="fred_sim_2dsensor_cam">-->
+<!--    <gazebo reference="mono_camera_link">-->
+<!--      <sensor type="camera" name="mono_camera">-->
+<!--        <update_rate>30.0</update_rate>-->
+<!--        <camera name="head">-->
+<!--          <horizontal_fov>${90.0*M_PI/180.0}</horizontal_fov>-->
+<!--          <image>-->
+<!--            <width>1280</width>-->
+<!--            <height>720</height>-->
+<!--            <format>R8G8B8</format>-->
+<!--          </image>-->
+<!--          <clip>-->
+<!--            <near>0.02</near>-->
+<!--            <far>30</far>-->
+<!--          </clip>-->
+<!--          <noise>-->
+<!--            <type>gaussian</type>-->
+<!--            &lt;!&ndash; Noise is sampled independently per pixel on each frame.-->
+<!--                That pixel's noise value is added to each of its color-->
+<!--                channels, which at that point lie in the range [0,1]. &ndash;&gt;-->
+<!--            <mean>0.0</mean>-->
+<!--            <stddev>0.007</stddev>-->
+<!--          </noise>-->
+<!--        </camera>-->
+<!--        <plugin name="camera_controller" filename="libgazebo_ros_camera.so">-->
+<!--          <alwaysOn>true</alwaysOn>-->
+<!--          <updateRate>0.0</updateRate>-->
+<!--          <cameraName>usb_cam</cameraName>-->
+<!--          <imageTopicName>image_raw</imageTopicName>-->
+<!--          <cameraInfoTopicName>camera_info</cameraInfoTopicName>-->
+<!--          <frameName>mono_camera_optical_frame</frameName>-->
+<!--          &lt;!&ndash; setting hackBaseline to anything but 0.0 will cause a misalignment-->
+<!--              between the gazebo sensor image and the frame it is supposed to-->
+<!--              be attached to &ndash;&gt;-->
+<!--          <hackBaseline>0.07</hackBaseline>-->
+<!--          <distortionK1>0.0</distortionK1>-->
+<!--          <distortionK2>0.0</distortionK2>-->
+<!--          <distortionK3>0.0</distortionK3>-->
+<!--          <distortionT1>0.0</distortionT1>-->
+<!--          <distortionT2>0.0</distortionT2>-->
+<!--          <CxPrime>0</CxPrime>-->
+<!--          <Cx>0.0</Cx>-->
+<!--          <Cy>0.0</Cy>-->
+<!--          <focalLength>0</focalLength>-->
+<!--        </plugin>-->
+<!--      </sensor>-->
+<!--    </gazebo>-->
+<!--  </xacro:macro>-->
   <xacro:macro name="fred_sim_2dsensor">
     <gazebo reference="hokuyo_link">

File: urdf/fred/fred_properties.urdf.xacro (robot description, xacro)
@@ -25,5 +25,23 @@
   <xacro:property name="cam_op" value="${M_PI/2}"/>
   <xacro:property name="cam_oy" value="0"/>
-  <!--
+    <!--
+   ======================================================================
+   - REP 119 : Monocular camera link relative to the Base link
+   ======================================================================
+     Base link is currently defined as the rotational centre on the bottom
+     of the base mould. For both create and kobuki this is actually exactly
+     the same 3d world point.
+     This may cause an issue with a base with much different floor clearance.
+     Should we be using base_footprint for this specification instead?
+     Note: REP needs to be updated with the information below
+     (currently in development and awaiting feedback)
+   -->
+	<xacro:property name="mono_cam_px" value="0.68" />
+<!--	<xacro:property name="cam_py" value="-0.0125" /> Y varies for different configurations. get sets in sensors_urdf -->
+	<xacro:property name="mono_cam_pz" value="0.11" />
+  <xacro:property name="mono_cam_or" value="0"/>
+  <xacro:property name="mono_cam_op" value="0"/>
+  <xacro:property name="mono_cam_oy" value="0"/>
+    <!--
   ======================================================================
   - REP 119 : Hokuyo laser link relative to the Base link
